File: pcb/encoder.kicad_pcb (KiCad board)
At the start: 2 copper layers, 32 x 57 mm, 2 parts, among them SW1 RKJXT1F42001, U1 Xiao2040

Commit message: fix pcb manually
Connections:
- U1 pad 1: SW_A -> ENC_B
- U1 pad 4: SW_D -> SW_PUSH
- U1 pad 5: SW_PUSH -> SW_A
- U1 pad 7: ENC_B -> SW_D
Routing:
- net SW_A: track 61.3 -> 32.8 mm, vias 2 -> 0
- net SW_D: track 30.6 -> 16.0 mm, vias 1 -> 0
- net SW_PUSH: track 49.9 -> 35.5 mm, vias 1 -> 0
- net SW_B: track 47.0 -> 38.0 mm
- net SW_C: track 28.9 -> 23.5 mm
- net ENC_A: track 25.8 -> 22.8 mm
- net ENC_B: track 37.7 -> 37.5 mm, vias 1 -> 0
- removed copper zone on B.Cu, net GND
Other:
- board outline removed

Commit message: fix pcb and firm
Parts:
- added REF**: screwhole, Suzuki:screwhole, F.Cu at (108.8, 108.0)
- added REF**: screwhole, Suzuki:screwhole, F.Cu at (91.5, 108.0)
Changed lines of the file:
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@@
+		(embedded_fonts no)
+	)
+	(footprint "Suzuki:screwhole"
+		(layer "F.Cu")
+		(at 108.75 108)
+		(property "Reference" "REF**"
+			(at 0 -2 0)
+			(unlocked yes)
+			(layer "F.SilkS")
+			(hide yes)
+			(effects
+				(font
+					(size 1 1)
+					(thickness 0.1)
+				)
+			)
+		)
+		(property "Value" "screwhole"
+			(at 0 2.8 0)
+			(unlocked yes)
+			(layer "F.Fab")
+			(hide yes)
+			(effects
+				(font
+					(size 1 1)
+					(thickness 0.15)
+				)
+			)
+		)
+		(property "Datasheet" ""
+			(at 0 0 0)
+			(unlocked yes)
+			(layer "F.Fab")
+			(hide yes)
+			(effects
+				(font
+					(size 1 1)
+					(thickness 0.15)
+				)
+			)
+		)
+		(property "Description" ""
+			(at 0 0 0)
+			(unlocked yes)
+			(layer "F.Fab")
+			(hide yes)
+			(effects
+				(font
+					(size 1 1)
+					(thickness 0.15)
+				)
+			)
+		)
+		(attr through_hole)
+		(duplicate_pad_numbers_are_jumpers no)
+		(pad "" np_thru_hole circle
+			(at -0.25 0)
+			(size 2 2)
+			(drill 2)
+			(layers "*.Cu" "*.Mask")
+		)
+		(embedded_fonts no)
+	)
+	(footprint "Suzuki:screwhole"
+		(layer "F.Cu")
+		(at 91.5 108)
+		(property "Reference" "REF**"
+			(at 0 -2 0)
+			(unlocked yes)
+			(layer "F.SilkS")
+			(hide yes)
+			(effects
+				(font
+					(size 1 1)
+					(thickness 0.1)
+				)
+			)
+		)
+		(property "Value" "screwhole"
+			(at 0 2.8 0)
+			(unlocked yes)
+			(layer "F.Fab")
+			(hide yes)
+			(effects
+				(font
+					(size 1 1)
+					(thickness 0.15)
+				)
+			)
+		)
+		(property "Datasheet" ""
+			(at 0 0 0)
+			(unlocked yes)
+			(layer "F.Fab")
+			(hide yes)
+			(effects
+				(font
+					(size 1 1)
+					(thickness 0.15)
+				)
+			)
+		)
+		(property "Description" ""
+			(at 0 0 0)
+			(unlocked yes)
+			(layer "F.Fab")
+			(hide yes)
+			(effects
+				(font
+					(size 1 1)
+					(thickness 0.15)
+				)
+			)
+		)
+		(attr through_hole)
+		(duplicate_pad_numbers_are_jumpers no)
+		(pad "" np_thru_hole circle
+			(at 0 0)
+			(size 2 2)
+			(drill 2)
+			(layers "*.Cu" "*.Mask")
+		)
 		(embedded_fonts no)
 	)
@@
 		(embedded_fonts no)
 	)
+	(gr_line
+		(start 89.5 65.5)
+		(end 89.5 109)
+		(stroke
+			(width 0.1)
+			(type solid)
+		)
+		(layer "F.SilkS")
+	)
+	(gr_arc
+		(start 89.5 65.5)
+		(mid 89.792893 64.792893)
+		(end 90.5 64.5)
+		(stroke
+			(width 0.1)
+			(type default)
+		)
+		(layer "F.SilkS")
+	)
+	(gr_line
+		(start 90.5 64.5)
+		(end 109.5 64.5)
+		(stroke
+			(width 0.1)
+			(type solid)
+		)
+		(layer "F.SilkS")
+	)
+	(gr_arc
+		(start 90.5 110)
+		(mid 89.792893 109.707107)
+		(end 89.5 109)
+		(stroke
+			(width 0.1)
+			(type default)
+		)
+		(layer "F.SilkS")
+	)
+	(gr_line
+		(start 90.5 110)
+		(end 109.5 110)
+		(stroke
+			(width 0.1)
+			(type solid)
+		)
+		(layer "F.SilkS")
+	)
+	(gr_arc
+		(start 109.5 64.5)
+		(mid 110.207107 64.792893)
+		(end 110.5 65.5)
+		(stroke
+			(width 0.1)
+			(type default)
+		)
+		(layer "F.SilkS")
+	)
+	(gr_line
+		(start 110.5 65.5)
+		(end 110.5 109)
+		(stroke
+			(width 0.1)
+			(type solid)
+		)
+		(layer "F.SilkS")
+	)
+	(gr_arc
+		(start 110.5 109)
+		(mid 110.207107 109.707107)
+		(end 109.5 110)
+		(stroke
+			(width 0.1)
+			(type default)
+		)
+		(layer "F.SilkS")
+	)
 	(segment

Commit message: fixpcb
Other:
- board outline added: 21 x 45.5 mm
Changed lines of the file:
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@@
 		(pad "Com" thru_hole circle
 			(at -1 -5.78)
-			(size 1.3 1.3)
+			(size 1.6 1.6)
 			(drill 0.8)
 			(layers "*.Cu" "*.Mask")
@@
 		(pad "ECom" thru_hole circle
 			(at -1.5 -7.8)
-			(size 1.4 1.4)
+			(size 1.6 1.6)
 			(drill 0.8)
 			(layers "*.Cu" "*.Mask")
@@
 			(type solid)
 		)
-		(layer "F.SilkS")
+		(layer "Edge.Cuts")
 	)
 	(gr_arc
@@
 			(type default)
 		)
-		(layer "F.SilkS")
+		(layer "Edge.Cuts")
 	)
 	(gr_line
@@
 			(type solid)
 		)
-		(layer "F.SilkS")
+		(layer "Edge.Cuts")
 	)
 	(gr_arc
@@
 			(type default)
 		)
-		(layer "F.SilkS")
+		(layer "Edge.Cuts")
 	)
 	(gr_line
@@
 			(type solid)
 		)
-		(layer "F.SilkS")
+		(layer "Edge.Cuts")
 	)
 	(gr_arc
@@
 			(type default)
 		)
-		(layer "F.SilkS")
+		(layer "Edge.Cuts")
 	)
 	(gr_line
@@
 			(type solid)
 		)
-		(layer "F.SilkS")
+		(layer "Edge.Cuts")
 	)
 	(gr_arc
@@
 			(type default)
 		)
-		(layer "F.SilkS")
+		(layer "Edge.Cuts")
+	)
+	(segment
+		(start 105.3 80.3)
+		(end 105.3 82.9)
+		(width 0.5)
+		(layer "B.Cu")
+		(net "ENC_B")
+	)
+	(segment
+		(start 92.38 67.38)
+		(end 105.3 80.3)
+		(width 0.5)
+		(layer "B.Cu")
+		(net "ENC_B")
+	)
+	(segment
+		(start 105.3 82.9)
+		(end 107.8 85.4)
+		(width 0.5)
+		(layer "B.Cu")
+		(net "ENC_B")
+	)
+	(segment
+		(start 107.8 85.4)
+		(end 107.8 98.5)
+		(width 0.5)
+		(layer "B.Cu")
+		(net "ENC_B")
+	)
+	(segment
+		(start 92.38 69.92)
+		(end 104 81.54)
+		(width 0.5)
+		(layer "B.Cu")
+		(net "SW_B")
+	)
+	(segment
+		(start 104 97.7)
+		(end 107.8 101.5)
+		(width 0.5)
+		(layer "B.Cu")
+		(net "SW_B")
+	)
+	(segment
+		(start 104 81.54)
+		(end 104 97.7)
+		(width 0.5)
+		(layer "B.Cu")
+		(net "SW_B")
+	)
+	(segment
+		(start 101.5 81.58)
+		(end 101.5 92.2)
+		(width 0.5)
+		(layer "B.Cu")
+		(net "SW_C")
+	)
+	(segment
+		(start 92.38 72.46)
+		(end 101.5 81.58)
+		(width 0.5)
+		(layer "B.Cu")
+		(net "SW_C")
+	)
+	(segment
+		(start 95.75 97.25)
+		(end 101 102.5)
+		(width 0.5)
+		(layer "B.Cu")
+		(net "SW_PUSH")
+	)
+	(segment
+		(start 92.38 75.04)
+		(end 95.75 78.41)
+		(width 0.5)
+		(layer "B.Cu")
+		(net "SW_PUSH")
+	)
+	(segment
+		(start 95.75 78.41)
+		(end 95.75 97.25)
+		(width 0.5)
+		(layer "B.Cu")
+		(net "SW_PUSH")
+	)
+	(segment
+		(start 101 102.5)
+		(end 101 106.98)
+		(width 0.5)
+		(layer "B.Cu")
+		(net "SW_PUSH")
 	)
 	(segment
@@
 	)
 	(segment
-		(start 104.3 81.84)
-		(end 104.3 98)
-		(width 0.5)
-		(layer "B.Cu")
-		(net "SW_B")
-	)
-	(segment
-		(start 92.38 69.92)
-		(end 104.3 81.84)
-		(width 0.5)
-		(layer "B.Cu")
-		(net "SW_B")
-	)
-	(segment
-		(start 104.3 98)
-		(end 107.8 101.5)
-		(width 0.5)
-		(layer "B.Cu")
-		(net "SW_B")
-	)
-	(segment
-		(start 101.5 81.58)
-		(end 101.5 92.2)
-		(width 0.5)
-		(layer "B.Cu")
-		(net "SW_C")
-	)
-	(segment
-		(start 92.38 72.46)
-		(end 101.5 81.58)
-		(width 0.5)
-		(layer "B.Cu")
-		(net "SW_C")
+		(start 92.38 80.08)
+		(end 90.6 81.86)
+		(width 0.5)
+		(layer "B.Cu")
+		(net "ENC_A")
+	)
+	(segment
+		(start 90.6 81.86)
+		(end 90.6 99.9)
+		(width 0.5)
+		(layer "B.Cu")
+		(net "ENC_A")
+	)
+	(segment
+		(start 90.6 99.9)
+		(end 92.2 101.5)
+		(width 0.5)
+		(layer "B.Cu")
+		(net "ENC_A")
 	)
 	(segment
@@
 	)
 	(segment
-		(start 101 102.9)
-		(end 101 106.98)
-		(width 0.5)
-		(layer "B.Cu")
-		(net "SW_PUSH")
-	)
-	(segment
-		(start 97.05 79.71)
-		(end 97.05 98.95)
-		(width 0.5)
-		(layer "B.Cu")
-		(net "SW_PUSH")
-	)
-	(segment
-		(start 92.38 75.04)
-		(end 97.05 79.71)
-		(width 0.5)
-		(layer "B.Cu")
-		(net "SW_PUSH")
-	)
-	(segment
-		(start 97.05 98.95)
-		(end 101 102.9)
-		(width 0.5)
-		(layer "B.Cu")
-		(net "SW_PUSH")
-	)
-	(segment
-		(start 92.38 80.08)
-		(end 90.6 81.86)
-		(width 0.5)
-		(layer "B.Cu")
-		(net "ENC_A")
-	)
-	(segment
-		(start 90.6 81.86)
-		(end 90.6 99.9)
-		(width 0.5)
-		(layer "B.Cu")
-		(net "ENC_A")
-	)
-	(segment
-		(start 90.6 99.9)
-		(end 92.2 101.5)
-		(width 0.5)
-		(layer "B.Cu")
-		(net "ENC_A")
-	)
-	(segment
-		(start 105.3 80.3)
-		(end 105.3 82.9)
-		(width 0.5)
-		(layer "B.Cu")
-		(net "ENC_B")
-	)
-	(segment
-		(start 92.38 67.38)
-		(end 105.3 80.3)
-		(width 0.5)
-		(layer "B.Cu")
-		(net "ENC_B")
-	)
-	(segment
-		(start 105.3 82.9)
-		(end 107.8 85.4)
-		(width 0.5)
-		(layer "B.Cu")
-		(net "ENC_B")
-	)
-	(segment
-		(start 107.8 85.4)
-		(end 107.8 98.5)
-		(width 0.5)
-		(layer "B.Cu")
-		(net "ENC_B")
-	)
-	(segment
 		(start 99 94.22)
 		(end 99 97.7)
@@
 	)
 	(segment
+		(start 109.37 102.37137)
+		(end 107.99137 103.75)
+		(width 0.5)
+		(layer "B.Cu")
+		(net "GND")
+	)
+	(segment
+		(start 107.99137 103.75)
+		(end 106.86 103.75)
+		(width 0.5)
+		(layer "B.Cu")
+		(net "GND")
+	)
+	(segment
+		(start 99 97.7)
+		(end 105.05 103.75)
+		(width 0.5)
+		(layer "B.Cu")
+		(net "GND")
+	)
+	(segment
 		(start 98.5 93.72)
 		(end 99 94.22)
 		(width 0.5)
 		(layer "B.Cu")
-		(net "GND")
-	)
-	(segment
-		(start 109.37 102.37137)
-		(end 107.99137 103.75)
-		(width 0.5)
-		(layer "B.Cu")
-		(net "GND")
-	)
-	(segment
-		(start 107.99137 103.75)
-		(end 106.86 103.75)
-		(width 0.5)
-		(layer "B.Cu")
-		(net "GND")
-	)
-	(segment
-		(start 99 97.7)
-		(end 105.05 103.75)
-		(width 0.5)
-		(layer "B.Cu")
